File: imu-harvester.kicad_pcb (KiCad board)
At the start: 4 copper layers, 48 x 15 mm, 59 parts, among them J1 53261-0671, J2 53261-0671, Q1 CSD23381F4, SW1 SLW-913535-2A-RA-D, T1 1:100, T2 1:100, U1 LTC3109EUF-PBF, U2 2450AT18A100E, U3 nRF52811-QCxx, U4 TPS7A0222PDBVR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

Commit message: route
Parts:
- removed TP5: +VST, TestPoint:TestPoint_Pad_D1.0mm
- removed TP6: -VST, TestPoint:TestPoint_Pad_D1.0mm
- TP7, TP8: moved to F.Cu
- moved TP13 26.4 mm to (210.0, 57.3), turned to 90 degrees
- moved TP14 24.0 mm to (211.4, 57.3), turned to 90 degrees
- moved TP11 21.0 mm to (207.2, 57.3), turned to -90 degrees
- moved TP12 20.8 mm to (208.6, 57.3), turned to 90 degrees
- moved TP9 18.5 mm to (200.3, 50.8), turned to -90 degrees
- moved TP10 15.4 mm to (201.7, 50.8), turned to -90 degrees
- moved TP8 13.2 mm to (190.7, 55.7), turned to 0 degrees
- moved TP7 11.2 mm to (196.9, 55.7), turned to 0 degrees
- moved C24 5.50 mm to (182.0, 49.0)
- moved C25 1.50 mm to (182.0, 54.0)
- moved R3 1.50 mm to (182.0, 55.0)
- moved TP1 0.40 mm to (185.1, 55.0)
- moved TP2 0.40 mm to (186.6, 57.5)
- moved TP3 0.40 mm to (188.1, 55.0)
- moved TP4 0.40 mm to (189.6, 57.5)
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Routing:
- net GND: track 0.00 -> 29.2 mm, vias 0 -> 36
- net /IMU_INT2: track 0.00 -> 16.1 mm, vias 0 -> 1
- net /~{IMU_CS}: track 0.00 -> 14.6 mm, vias 0 -> 1
- net /DIV_EN: track 0.00 -> 14.1 mm, vias 0 -> 2
- net /V_STORE_DIV: track 0.00 -> 14.0 mm, vias 0 -> 2
- net /IMU_SCK: track 0.00 -> 13.7 mm, vias 0 -> 1
- net /IMU_INT1: track 0.00 -> 13.7 mm, vias 0 -> 1
- net /-V_Stator: track 0.00 -> 13.3 mm, vias 0 -> 2
- net /IMU_MOSI: track 0.00 -> 11.9 mm, vias 0 -> 1
- net /SWDCLK: track 0.00 -> 10.3 mm, vias 0 -> 2
- net /IMU_MISO: track 0.00 -> 9.97 mm, vias 0 -> 1
- net /SWDIO: track 0.00 -> 9.80 mm, vias 0 -> 2
- net Net-(D1-K): track 0.00 -> 9.02 mm, vias 0 -> 1
- net +3V3: track 0.00 -> 8.87 mm, vias 0 -> 8
- net /LTC_VAUX: track 0.00 -> 8.52 mm, vias 0 -> 2
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- added copper zone on B.Cu, net +3V3
- added copper zone on F.Cu, net +3V3
- added copper zone on In2.Cu, net +3V3
- added copper zone on F.Cu, net /+V_Stator
- added copper zone on F.Cu, net /-V_Stator
- added copper zone on F.Cu, net /ANT
- added copper zone on B.Cu, net /LTC_SWA
- added copper zone on B.Cu, net /LTC_SWB
- added copper zone on B.Cu, net /VDD_Ext
- added copper zone on F.Cu, net /VDD_Gen
- added copper zone on In2.Cu, net /VDD_Gen
- added copper zone on B.Cu, net /V_STORE
- added copper zone on F.Cu, net /V_STORE
- added copper zone on In2.Cu, net Net-(C12-Pad1)
- added copper zone on In2.Cu, net Net-(C6-Pad1)
Other:
- board text added: "EXT"
- board text added: "GEN"
- board text added: "GND"
- board text added: "VDD"
