File: imu-harvester.kicad_pcb (KiCad board)
At the start: 4 copper layers, 48 x 15 mm, 57 parts, among them J1 53261-0671, J2 53261-0671, Q1 CSD23381F4, SW1 SLW-913535-2A-RA-D, T1 1:100, T2 1:100, U1 LTC3109EUF-PBF, U2 2450AT18A100E, U3 nRF52811-QCxx, U4 TPS7A0222PDBVR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

Commit message: gerbers 2
Routing:
- net GND: vias 36 -> 41
Changed lines of the file:
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@@
       (stroke (width 0.05) (type solid)) (fill none) (layer "F.CrtYd"))
     (pad "1" smd circle (at 0 0) (size 1 1) (layers "F.Cu" "F.Mask")
-      (net 24 "/V_STORE") (pinfunction "1") (pintype "passive"))
+      (net 24 "/V_STORE") (pinfunction "1") (pintype "passive") (zone_connect 2))
   )
   (footprint "Capacitor_Tantalum_SMD:CP_EIA-6032-28_Kemet-C" (layer "F.Cu")
@@
       (stroke (width 0.05) (type solid)) (fill none) (layer "F.CrtYd"))
     (pad "1" smd circle (at 0 0) (size 1 1) (layers "F.Cu" "F.Mask")
-      (net 13 "/VDD_Gen") (pinfunction "1") (pintype "passive"))
+      (net 13 "/VDD_Gen") (pinfunction "1") (pintype "passive") (zone_connect 2))
   )
   (footprint "LED_SMD:LED_0603_1608Metric" (layer "F.Cu")
@@
   (segment (start 220.1 51.8) (end 219.5 51.2) (width 0.4) (layer "F.Cu") (net 7))
   (segment (start 219.025 58.125) (end 219 58.1) (width 0.4) (layer "F.Cu") (net 7))
+  (via (at 178 51) (size 0.5) (drill 0.3) (layers "F.Cu" "B.Cu") (free) (net 7))
   (via (at 217.5 57) (size 0.5) (drill 0.3) (layers "F.Cu" "B.Cu") (free) (net 7))
   (via (at 214.6 53.5) (size 0.5) (drill 0.3) (layers "F.Cu" "B.Cu") (net 7))
+  (via (at 178 57) (size 0.5) (drill 0.3) (layers "F.Cu" "B.Cu") (free) (net 7))
   (via (at 210.8 58.5) (size 0.5) (drill 0.3) (layers "F.Cu" "B.Cu") (free) (net 7))
   (via (at 190.6 54.4) (size 0.5) (drill 0.3) (layers "F.Cu" "B.Cu") (net 7))
   (via (at 217.5 60) (size 0.5) (drill 0.3) (layers "F.Cu" "B.Cu") (free) (net 7))
+  (via (at 178 59) (size 0.5) (drill 0.3) (layers "F.Cu" "B.Cu") (free) (net 7))
   (via (at 206.02 59.6) (size 0.5) (drill 0.3) (layers "F.Cu" "B.Cu") (net 7))
   (via (at 219 58.1) (size 0.5) (drill 0.3) (layers "F.Cu" "B.Cu") (net 7))
@@
   (via (at 205 50.2) (size 0.5) (drill 0.3) (layers "F.Cu" "B.Cu") (net 7))
   (via (at 216.1 51) (size 0.5) (drill 0.3) (layers "F.Cu" "B.Cu") (net 7))
+  (via (at 178 53) (size 0.5) (drill 0.3) (layers "F.Cu" "B.Cu") (free) (net 7))
   (via (at 197.4 59.1) (size 0.5) (drill 0.3) (layers "F.Cu" "B.Cu") (net 7))
   (via (at 190.6 53.2) (size 0.5) (drill 0.3) (layers "F.Cu" "B.Cu") (net 7))
@@
   (via (at 221.2 58.1) (size 0.5) (drill 0.3) (layers "F.Cu" "B.Cu") (net 7))
   (via (at 187.6 53.1) (size 0.5) (drill 0.3) (layers "F.Cu" "B.Cu") (free) (net 7))
+  (via (at 178 55) (size 0.5) (drill 0.3) (layers "F.Cu" "B.Cu") (free) (net 7))
   (segment (start 216.2 51.9) (end 217 51.9) (width 0.2) (layer "B.Cu") (net 7))
   (segment (start 193.500001 50.499999) (end 192.5 51.5) (width 0.2) (layer "B.Cu") (net 7))
