File: imu-harvester.kicad_sch (KiCad schematic)
At the start: 34 parts, among them J2 503480-0800, SW1 SW_SPDT, U1 2450AT18A100E, U2 LTC3109EUF-PBF, U3 nRF52811-QCxx, U4 TPS7A0222PDBVR, X1 32MHz, X2 32.768kHz

Commit message: schematic done
Parts:
- added C16: 10nF, Capacitor_SMD:C_0402_1005Metric, symbol Device:C_Small
- added C17: 470uF, symbol Device:C_Polarized
- added C18: ?, symbol Device:C_Polarized
- added C19, C21: 1nF, Capacitor_SMD:C_0402_1005Metric, symbol Device:C_Small
- added C20, C22: 470pF, Capacitor_SMD:C_0402_1005Metric, symbol Device:C_Small
- added C23: 1uF, Capacitor_SMD:C_0402_1005Metric, symbol Device:C_Small
- added C24: 2.2uF, Capacitor_SMD:C_0402_1005Metric, symbol Device:C_Small
- added Q1: Q_PMOS_DGS, symbol Device:Q_PMOS_DGS
- added R2: 10M, Resistor_SMD:R_0402_1005Metric, symbol Device:R_Small
- added R3: 5M, Resistor_SMD:R_0402_1005Metric, symbol Device:R_Small
- added T1, T2: 1:100, symbol Device:Transformer_1P_1S
- R1: footprint (none) -> Resistor_SMD:R_0402_1005Metric
Connections:
- net +V_Stator: now also U2.13 (VINB), T2.1 (AA)
- net -V_Stator: now also U2.14 (VINA), T1.1 (AA)
- net GND: now also U2.11 (GND), U2.16 (GND), U2.21 (EPAD), U2.8 (GND), C16.2, C17.2, C18.2, C23.2, C24.2, R3.2, T1.3 (SA), T2.3 (SA)
- net VDD: now also U2.7 (VLDO), C24.1
- net V_STORE: now reaches U2.1 (VSTORE)
- net V_STORE: now also C17.1, C18.1, Q1.1 (D)
- net LTC_C2B: now reaches U2.10 (C2B)
- net LTC_C2B: now also C20.2
- net LTC_SWB: now reaches U2.12 (SWB)
- net LTC_SWB: now also T1.2 (AB)
- net LTC_SWA: now reaches U2.15 (SWA)
- net LTC_SWA: now also T2.2 (AB)
- net LTC_C2A: now reaches U2.17 (C2A)
- net LTC_C2A: now also C22.2
- net LTC_C1A: now reaches U2.18 (C1A)
- net LTC_C1A: now also C21.2
- net LTC_VAUX: now reaches U2.19 (VS1)
- net LTC_VAUX: now also U2.2 (VAUX), U2.20 (VS2), C23.1
- net LTC_C1B: now reaches U2.9 (C1B)
- net LTC_C1B: now also C19.2
- net V_STORE_DIV: now reaches U3.4 (AIN2/P0.04)
- net V_STORE_DIV: now also C16.1, R2.1, R3.1
- net DIV_EN: now reaches U3.5 (AIN3/P0.05)
- net DIV_EN: now also Q1.2 (G)
- new net: C21.1, C22.1, T2.4 (SB)
- new net: Q1.3 (S), R2.2
- new net: C19.1, C20.1, T1.4 (SB)
- no-connect marks 12 -> 14
Other:
- note added: "Energy Harvester IC"
- note added: "Energy Storage Measurement"
- note added: "IMU"
- note added: "Power Source Switching"
- note added: "TODO: change JTAG connector? calculate required energy / find large caps"
- note added: "V_CAP_DIV = V_CAP / 3 V_CAP max = 5.25V"
- moved on the sheet: AC1, C1, C2, U2, U3

Commit message: big cap and transformer
Parts:
- removed T1, T2: 1:100, symbol Device:Transformer_1P_1S
- added C25: ?, symbol Device:C_Polarized
- added T1, T3: 1:100, E-Tattoo_Parts:74488540070, symbol E-Tattoo_Parts:74488540070
- C17: value 470uF -> 100uF; footprint (none) -> Capacitor_Tantalum_SMD:CP_EIA-6032-28_Kemet-C
Connections:
- net +V_Stator: now also T3.1
- net -V_Stator: now also T1.1
- net GND: now also C25.2, T1.3, T3.3
- net LTC_SWA: now also T3.2
- net LTC_SWB: now also T1.2
- net V_STORE: now also C25.1
- net at C21.1, C22.1: now also T3.4
- net at C19.1, C20.1: now also T1.4
Other:
- note added: "Energy per capacitor 0.5 * 100uF * (5.25V)^2 = 1.380mJ"
- note removed: "TODO: change JTAG connector? calculate required energy / find large caps"
- moved on the sheet: C17, C18, C19, C20, C21, C22, C23, C24

Commit message: parts
Parts:
- removed J1: ~, symbol E-Tattoo_Parts:SWD-Connector
- removed J2: 503480-0800, E-Tattoo_Parts:503480-0800, symbol E-Tattoo_Parts:503480-0800
- removed Q1: Q_PMOS_DGS, symbol Device:Q_PMOS_DGS
- added J1, J2: 53261-0671, E-Tattoo_Parts:532610671, symbol E-Tattoo_Parts:53261-0671
- added Q2: CSD23381F4, E-Tattoo_Parts:CSD23381F4, symbol E-Tattoo_Parts:CSD23381F4
- C1, C10, C11, C2, C9: Dielectric (none) -> X7R; Manufacturer_Part_Number (none) -> KGM05AR71C104KN
- C12: Dielectric (none) -> NP0; Manufacturer_Part_Number (none) -> KGM05ACG1H101JN
- C13, C14, C15, C23: Dielectric (none) -> X7R; Manufacturer_Part_Number (none) -> CM05X7R105K06AH-HE
- C16: Dielectric (none) -> X7R; Manufacturer_Part_Number (none) -> C0402C103K1RACAUTO
- C17: Manufacturer_Part_Number (none) -> TL3C107K010C0200
- C19, C21: Dielectric (none) -> X7R; Manufacturer_Part_Number (none) -> C0402C102KCRACAUTO
- C20, C22: Dielectric (none) -> NP0; Manufacturer_Part_Number (none) -> KGM05ACG1H471JH
- C24: Dielectric (none) -> X7R; Manufacturer_Part_Number (none) -> GRM155Z71A225KE01D
- C3: Dielectric (none) -> NP0; Manufacturer_Part_Number (none) -> GRM1555C1ER80BA01D
- C4, C5, C6, C7: Dielectric (none) -> NP0; Manufacturer_Part_Number (none) -> KGM05ACG1H120JN
- C8: footprint Capacitor_SMD:C_0402_1005Metric -> Capacitor_SMD:C_0603_1608Metric; Dielectric (none) -> X7R; Manufacturer_Part_Number (none) -> GRM188Z71C475KE21D
- D1: Manufacturer_Part_Number (none) -> LO Q976.01-P2R2-25-1
- L1: Manufacturer_Part_Number (none) -> LQG15WZ3N9B02D
- L2: footprint Inductor_SMD:L_0402_1005Metric -> Inductor_SMD:L_0603_1608Metric; Manufacturer_Part_Number (none) -> KLZ1608MHR100WTD25
- L3: Manufacturer_Part_Number (none) -> LQG15WZ15NG02D
- R1: Manufacturer_Part_Number (none) -> RCC040210R0FKED
- R2: Manufacturer_Part_Number (none) -> RCC040210M0FKED
- R3: Manufacturer_Part_Number (none) -> CRCW04024M99FKED
- SW1: value SW_SPDT -> SLW-913535-2A-RA-D; footprint (none) -> E-Tattoo_Parts:SLW-913535-2A-RA-D; Height (none) -> 3.5; Manufacturer_Part_Number (none) -> SLW-913535-2A-RA-D
- T1, T3: Height (none) -> 4.0; Manufacturer_Part_Number (none) -> 74488540070
- U1: Manufacturer_Part_Number (none) -> 2450AT18A100E
- U2: Manufacturer_Part_Number (none) -> LTC3109EUF#PBF
- U3: Manufacturer_Part_Number (none) -> nRF52811-QCAA-R
- U4: Manufacturer_Part_Number (none) -> TPS7A0222PDBVR
- X1: footprint (none) -> Crystal:Crystal_SMD_2016-4Pin_2.0x1.6mm; Manufacturer_Part_Number (none) -> ECS-320-8-37B2-JTY-TR
- X2: footprint (none) -> Crystal:Crystal_SMD_2012-2Pin_2.0x1.2mm; symbol Device:Crystal_GND24 -> Device:Crystal; Manufacturer_Part_Number (none) -> ECS-.327-9-12R-TR
Connections:
- net +3V3: now also J2.5
- net +V_Stator: now also J1.1, J1.2, J1.3
- net -V_Stator: now also J1.4, J1.5, J1.6
- net DIV_EN: now also Q2.1 (G)
- net GND: now also J2.1, J2.6; no longer X2.2, X2.4
- net SWDCLK: now also J2.2
- net SWDIO: now also J2.3
- net VDD: now also J2.4; no longer C24.1, U2.7 (VLDO)
- net VDD_Gen: now also C24.1, U2.7 (VLDO)
- net V_STORE: now also Q2.2 (S)
- net XL1: now also X2.2; no longer X2.3
- net at R2.2: now also Q2.3 (D)
- no-connect marks 14 -> 18
Other:
- moved on the sheet: C16, C23, C24, R2, R3

Commit message: tps
Parts:
- added TP10: SCK, TestPoint:TestPoint_Pad_D2.0mm, symbol Connector:TestPoint
- added TP11: MISO, TestPoint:TestPoint_Pad_D2.0mm, symbol Connector:TestPoint
- added TP12: MOSI, TestPoint:TestPoint_Pad_D2.0mm, symbol Connector:TestPoint
- added TP13: INT1, TestPoint:TestPoint_Pad_D2.0mm, symbol Connector:TestPoint
- added TP14: INT2, TestPoint:TestPoint_Pad_D2.0mm, symbol Connector:TestPoint
- added TP5: +VST, TestPoint:TestPoint_Pad_D2.0mm, symbol Connector:TestPoint
- added TP6: -VST, TestPoint:TestPoint_Pad_D2.0mm, symbol Connector:TestPoint
- added TP7: VCAP, TestPoint:TestPoint_Pad_D2.0mm, symbol Connector:TestPoint
- added TP8: 2V2_Gen, TestPoint:TestPoint_Pad_D2.0mm, symbol Connector:TestPoint
- added TP9: CS, TestPoint:TestPoint_Pad_D2.0mm, symbol Connector:TestPoint
- C15: renamed from C18; footprint (none) -> Capacitor_Tantalum_SMD:CP_EIA-6032-28_Kemet-C
- C16: renamed from C25; footprint (none) -> Capacitor_Tantalum_SMD:CP_EIA-6032-28_Kemet-C
- TP1, TP2, TP3, TP4: footprint E-Tattoo_Parts:Testpoint_Hex_D1.5 -> E-Tattoo_Parts:Testpoint_Hex_D3.0
- renumbered C6 to C10, C7 to C11, C19 to C12, C20 to C13, C17 to C14, C8 to C17, C9 to C18, C10 to C19, C16 to C20, C11 to C21, C12 to C22, C13 to C23, C14 to C24, C15 to C25, C23 to C4, C24 to C5, C21 to C6, C22 to C7, C4 to C8, C5 to C9, Q2 to Q1, R2 to R1, R3 to R2, R1 to R3, T3 to T1, T1 to T2, U2 to U1, U1 to U2
Connections:
- net +V_Stator: now also TP5.1
- net -V_Stator: now also TP6.1
- net IMU_INT1: now also TP13.1
- net IMU_INT2: now also TP14.1
- net IMU_MISO: now also TP11.1
- net IMU_MOSI: now also TP12.1
- net IMU_SCK: now also TP10.1
- net VDD_Gen: now also TP8.1
- net V_STORE: now also TP7.1
- net ~{IMU_CS}: now also TP9.1
Other:
- moved on the sheet: U3

Commit message: place
Parts:
- TP10, TP11, TP12, TP13, TP14, TP5, TP6, TP7, TP8, TP9: footprint TestPoint:TestPoint_Pad_D2.0mm -> TestPoint:TestPoint_Pad_D1.0mm
Changed lines of the file:
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@@
       (effects (font (size 1.27 1.27)) (justify left))
     )
-    (property "Footprint" "TestPoint:TestPoint_Pad_D2.0mm" (at 109.22 94.615 0)
+    (property "Footprint" "TestPoint:TestPoint_Pad_D1.0mm" (at 109.22 94.615 0)
       (effects (font (size 1.27 1.27)) hide)
     )
@@
       (effects (font (size 1.27 1.27)) (justify left))
     )
-    (property "Footprint" "TestPoint:TestPoint_Pad_D2.0mm" (at 106.045 69.85 0)
+    (property "Footprint" "TestPoint:TestPoint_Pad_D1.0mm" (at 106.045 69.85 0)
       (effects (font (size 1.27 1.27)) hide)
     )
@@
       (effects (font (size 1.27 1.27)) (justify left))
     )
-    (property "Footprint" "TestPoint:TestPoint_Pad_D2.0mm" (at 193.675 125.095 0)
+    (property "Footprint" "TestPoint:TestPoint_Pad_D1.0mm" (at 193.675 125.095 0)
       (effects (font (size 1.27 1.27)) hide)
     )
@@
       (effects (font (size 1.27 1.27)) (justify left))
     )
-    (property "Footprint" "TestPoint:TestPoint_Pad_D2.0mm" (at 193.675 122.555 0)
+    (property "Footprint" "TestPoint:TestPoint_Pad_D1.0mm" (at 193.675 122.555 0)
       (effects (font (size 1.27 1.27)) hide)
     )
@@
       (effects (font (size 1.27 1.27)) (justify left))
     )
-    (property "Footprint" "TestPoint:TestPoint_Pad_D2.0mm" (at 193.675 127.635 0)
+    (property "Footprint" "TestPoint:TestPoint_Pad_D1.0mm" (at 193.675 127.635 0)
       (effects (font (size 1.27 1.27)) hide)
     )
@@
       (effects (font (size 1.27 1.27)) (justify left))
     )
-    (property "Footprint" "TestPoint:TestPoint_Pad_D2.0mm" (at 193.675 117.475 0)
+    (property "Footprint" "TestPoint:TestPoint_Pad_D1.0mm" (at 193.675 117.475 0)
       (effects (font (size 1.27 1.27)) hide)
     )
@@
       (effects (font (size 1.27 1.27)) (justify left))
     )
-    (property "Footprint" "TestPoint:TestPoint_Pad_D2.0mm" (at 45.72 76.835 0)
+    (property "Footprint" "TestPoint:TestPoint_Pad_D1.0mm" (at 45.72 76.835 0)
       (effects (font (size 1.27 1.27)) hide)
     )
@@
       (effects (font (size 1.27 1.27)) (justify left))
     )
-    (property "Footprint" "TestPoint:TestPoint_Pad_D2.0mm" (at 193.675 114.935 0)
+    (property "Footprint" "TestPoint:TestPoint_Pad_D1.0mm" (at 193.675 114.935 0)
       (effects (font (size 1.27 1.27)) hide)
     )
@@
       (effects (font (size 1.27 1.27)) (justify left))
     )
-    (property "Footprint" "TestPoint:TestPoint_Pad_D2.0mm" (at 193.675 120.015 0)
+    (property "Footprint" "TestPoint:TestPoint_Pad_D1.0mm" (at 193.675 120.015 0)
       (effects (font (size 1.27 1.27)) hide)
     )
@@
       (effects (font (size 1.27 1.27)) (justify left))
     )
-    (property "Footprint" "TestPoint:TestPoint_Pad_D2.0mm" (at 45.72 97.155 0)
-      (effects (font (size 1.27 1.27)) hide)
-    )
+    (property "Footprint" "TestPoint:TestPoint_Pad_D1.0mm" (at 45.72 97.155 0)
+      (effects (font (size 1.27 1.27)) hide)
+    )

Commit message: route
Parts:
- removed TP5: +VST, TestPoint:TestPoint_Pad_D1.0mm, symbol Connector:TestPoint
- removed TP6: -VST, TestPoint:TestPoint_Pad_D1.0mm, symbol Connector:TestPoint
Changed lines of the file:
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@@
   (junction (at 40.64 182.245) (diameter 0) (color 0 0 0 0)
   )
-  (junction (at 40.64 76.835) (diameter 0) (color 0 0 0 0)
-  )
   (junction (at 100.965 69.85) (diameter 0) (color 0 0 0 0)
   )
@@
   (junction (at 51.435 97.155) (diameter 0) (color 0 0 0 0)
   )
-  (junction (at 40.64 97.155) (diameter 0) (color 0 0 0 0)
-  )
   (junction (at 31.115 174.625) (diameter 0) (color 0 0 0 0)
   )
@@
     )
   )
-  (symbol (lib_id "Connector:TestPoint") (at 40.64 76.835 0) (unit 1)
-    (in_bom no) (on_board yes) (dnp no) (fields_autoplaced)
-    (property "Reference" "TP5" (at 43.18 72.898 0)
-      (effects (font (size 1.27 1.27)) (justify left))
-    )
-    (property "Value" "+VST" (at 43.18 75.438 0)
-      (effects (font (size 1.27 1.27)) (justify left))
-    )
-    (property "Footprint" "TestPoint:TestPoint_Pad_D1.0mm" (at 45.72 76.835 0)
-      (effects (font (size 1.27 1.27)) hide)
-    )
-    (property "Datasheet" "~" (at 45.72 76.835 0)
-      (effects (font (size 1.27 1.27)) hide)
-    )
-    (pin "1")
-    (instances
-      (project "imu-harvester"
-        (path "/fece34dc-1cbe-4879-bbf7-9dbb0cf9798a"
-          (reference "TP5") (unit 1)
-        )
-      )
-    )
-  )
   (symbol (lib_id "power:VDD") (at 171.45 47.625 270) (unit 1)
     (in_bom yes) (on_board yes) (dnp no) (fields_autoplaced)
@@
         )
       )
-    )
-  )
-  (symbol (lib_id "Connector:TestPoint") (at 40.64 97.155 0) (unit 1)
-    (in_bom no) (on_board yes) (dnp no) (fields_autoplaced)
-    (property "Reference" "TP6" (at 43.18 93.218 0)
-      (effects (font (size 1.27 1.27)) (justify left))
-    )
-    (property "Value" "-VST" (at 43.18 95.758 0)
-      (effects (font (size 1.27 1.27)) (justify left))
-    )
-    (property "Footprint" "TestPoint:TestPoint_Pad_D1.0mm" (at 45.72 97.155 0)
-      (effects (font (size 1.27 1.27)) hide)
-    )
-    (property "Datasheet" "~" (at 45.72 97.155 0)
-      (effects (font (size 1.27 1.27)) hide)
-    )
-    (pin "1")
-    (instances
-      (project "imu-harvester"
-        (path "/fece34dc-1cbe-4879-bbf7-9dbb0cf9798a"
-          (reference "TP6") (unit 1)
-        )
-      )
